File: AIS-Converter.kicad_sch (KiCad schematic)
At the start: 0 parts

Commit message: Adding hierarchical blocks
Parts:
- added J1, J2, J3: 691216510002S, Wurth Git:J_Wurth_WR-TBL_691216510002S, symbol Wurth Git:691216510002S
- added J4: Raspberry_Pi_4, Connector_PinHeader_2.54mm:PinHeader_2x20_P2.54mm_Vertical, symbol Connector:Raspberry_Pi_4
- added J5: USB_C_Receptacle_USB2.0_14P, symbol Connector:USB_C_Receptacle_USB2.0_14P
- added J6, J7: Conn_Coaxial_Small, Rick:SMA-KWE_C7498154, symbol Connector:Conn_Coaxial_Small
Connections:
- new net: J5.A1 (GND), J5.A12 (GND), J5.B1 (GND), J5.B12 (GND)
- new net: J5.A4 (VBUS), J5.A9 (VBUS), J5.B4 (VBUS), J5.B9 (VBUS)
- new net: J4.1 (3V3), J4.17 (3V3)
- new net: J4.14 (GND), J4.20 (GND), J4.25 (GND), J4.30 (GND), J4.34 (GND), J4.39 (GND), J4.6 (GND), J4.9 (GND)
- new net: J4.2 (5V), J4.4 (5V)
- new net GND: J6.1 (Ext), J6.2 (Ext), J6.3 (Ext), J6.4 (Ext), J7.1 (Ext), J7.2 (Ext), J7.3 (Ext), J7.4 (Ext)
- new net Modem/GNSS_ANT: J7.5 (In)
- new net Modem/SIM_ANT: J6.5 (In)
Other:
- added sheet Ethernet PHY (ethernet.kicad_sch)
- added sheet Microcontroller (microcontroller.kicad_sch)
- added sheet Modem (modem.kicad_sch)
- added sheet Power (power.kicad_sch)

Commit message: progress save
Parts:
- removed J1, J2, J3: 691216510002S, Wurth Git:J_Wurth_WR-TBL_691216510002S, symbol Wurth Git:691216510002S
- added J1: Conn_01x02, Rick:J_Wurth_WR-TBL_691322110006, symbol Connector_Generic:Conn_01x02
