File: AIS-Converter.kicad_sch (KiCad schematic)
At the start: 5 parts, among them J1 Conn_01x02, J4 Raspberry_Pi_4, J5 USB_C_Receptacle_USB2.0_14P, J6 Conn_Coaxial_Small, J7 Conn_Coaxial_Small

Commit message: Adding ethernet module and more
Parts:
- removed J5: USB_C_Receptacle_USB2.0_14P, symbol Connector:USB_C_Receptacle_USB2.0_14P
- added J2: USB_C_Receptacle_USB2.0_16P, Connector_USB:USB_C_Receptacle_Amphenol_124019772112A, symbol Rick:USB_C_Receptacle_USB2.0_16P
- added J3: Conn_01x04, Rick:J_Wurth_WR-TBL_691322110004, symbol Connector_Generic:Conn_01x04
- added R1, R2: 5k1, Resistor_SMD:R_0805_2012Metric, symbol Device:R
- added U13: USBLC6-2SC6, Package_TO_SOT_SMD:SOT-23-6, symbol Power_Protection:USBLC6-2SC6
- added U3: dAISy-catcher, Rick:dAISy-catcher-11mm, symbol Rick:dAISy-catcher
- added U4: HY931147C, Rick:HY931147C, symbol Rick:HY931147C_new
- J1: footprint Rick:J_Wurth_WR-TBL_691322110006 -> Rick:J_Wurth_WR-TBL_691322110002
Connections:
- net Modem/SIM_ANT is gone; now on net ANT: J6.5 (In)
- net GND: now also J1.2 (Pin_2), J2.A1 (GND), J2.A12 (GND), J2.B1 (GND), J2.B12 (GND), R1.2, R2.2, U13.2 (GND), U4.GND1, U4.GND2
- net Power/VN_PoE: now also U4.V-
- net Power/VP12V: now also J1.1 (Pin_1)
- net Power/VP_PoE: now also U4.V+
- net Power/VP_USB: now also J2.A4 (VBUS), J2.A9 (VBUS), J2.B4 (VBUS), J2.B9 (VBUS), U13.5 (VBUS)
- net Modem/GNSS_ANT renamed ANT
- new net: J2.A5 (CC1), R2.1
- new net: J2.B5 (CC2), R1.1
- new net DN: J2.A7 (D-), J2.B7 (D-), U13.3 (I/O2)
- new net DP: J2.A6 (D+), J2.B6 (D+), U13.1 (I/O1)
- new net USB to Serial/USB_DN: U13.4 (I/O2)
- new net USB to Serial/USB_DP: U13.6 (I/O1)
- no-connect marks 0 -> 2
Other:
- added sheet USB to Serial (USB-Serial.kicad_sch)
- sheet Ethernet PHY ports: added 3V3, ETH_ACT_LED, ETH_LINK_LED, GND; removed none
- sheet Microcontroller ports: added CH_DTR, CH_RTS, ESP_RXD0, ESP_TXD0; removed none
- sheet Power ports: added none; removed VN_USB
- note added: "12VDC INPUT"
- note added: "5k1 (Request 5VDC)"
- note added: "ADD filtering to GPS"
- note added: "Check netclasses impedanc JLC calculator wastn matching with order stackup"
- moved on the sheet: J1, J4, J6, J7

Commit message: Ethernet progress, 40pin connector, save progress
Parts:
- added C19: 22n, Capacitor_SMD:C_0603_1608Metric, symbol Device:C
- added R35, R36: 1k5, Resistor_SMD:R_0603_1608Metric, symbol Device:R
- added R51, R52: 0R, Resistor_SMD:R_0603_1608Metric, symbol Device:R
- J4: value Raspberry_Pi_4 -> Raspberry_Pi_40pin_Connector; symbol Connector:Raspberry_Pi_4 -> Rick:Raspberry_Pi_4_Custom
- U3: now left out of the parts list
Connections:
- net Ethernet PHY/ETH_ACT_LED: now also R35.2
- net Ethernet PHY/ETH_LINK_LED: now also R36.2
- net GND: now also J4.14 (GND), J4.20 (GND), J4.25 (GND), J4.30 (GND), J4.34 (GND), J4.39 (GND), J4.6 (GND), J4.9 (GND), U4.Y-, C19.2
- net VP5V: now also J4.2 (5V), J4.4 (5V)
- net VDDA_3V3: now reaches U4.G+
- net VDDA_3V3: now also U4.RXCT, U4.TXCT, C19.1
- net at U4.G-: now also R36.1
- net Ethernet PHY/RXP: now reaches U4.RX+
- net Ethernet PHY/RXN: now reaches U4.RX-
- net Ethernet PHY/TXP: now reaches U4.TX+
- net Ethernet PHY/TXN: now reaches U4.TX-
- net at U4.Y+: now also R35.1
- net at J4.10 (GPIO15/UART_RXD): now also R52.1
- net at J4.8 (GPIO14/UART_TXD): now also R51.1
- new net Microcontroller/AIS_UART0_TX: R51.2
- new net Microcontroller/AIS_UART_RX: R52.2
- no-connect marks 2 -> 29
Other:
- sheet Ethernet PHY ports: added CRS_DV/MODE2, ETH_CLK, MDC, MDIO, RXD0/MODE0, RXD1/MODE1, RXER/PHYADD0, RXN, RXP, TXD0, TXD1, TXEN, TXN, TXP, VP3V3, VP3V3_VDDA; removed 3V3
- sheet Microcontroller ports: added AIS_UART0_TX, AIS_UART_RX, CRS_DV, ETH_CLK, MDC, MDIO, RXD0, RXD1, TXD0, TXD1, TXEN; removed none
- note added: "100ohm diff Z"
- note added: "100ohm single ended Z"
- note added: "Check 50ohm impedance for lte and gps JLC stackup JLC04161H-7628"
- note added: "Fred?"
- note added: "TODO: - POWER LEDs - USER LEDs - GPS ANTENNA MATCHING CIRCUIT - CAN DRIVER - NMEA 0183 - NMEA 2000 - M12 CONNECTOR - SCHEMATIC CHECK - TEST POINTS - MOUNTING HOLES - ??"
- note added: "check shield connection! split grounds"
- note added: "reverse polarity protection P fet and zener"
- note removed: "Check netclasses impedanc JLC calculator wastn matching with order stackup"
- moved on the sheet: J4, J6, J7

Commit message: NMEA0183 and NMEA2000 schematics
Parts:
- added J5: Conn_01x02, Connector_PinSocket_2.54mm:PinSocket_2x03_P2.54mm_Vertical, symbol Connector_Generic:Conn_01x06
- added J8: M12A-05PMMR-SF7003, Rick:M12A05PMMRSF7003, symbol Connector_Generic:Conn_01x05
- J3: value Conn_01x04 -> Conn_01x05; footprint Rick:J_Wurth_WR-TBL_691322110004 -> Rick:J_Wurth_WR-TBL_691322110005; symbol Connector_Generic:Conn_01x04 -> Connector_Generic:Conn_01x05
Connections:
- net GND: now also J3.5 (Pin_5), J5.6 (Pin_6), J8.1 (Pin_1)
- net NMEA0183/TXP: now reaches J3.1 (Pin_1)
- net NMEA0183/TXN: now reaches J3.2 (Pin_2)
- net NMEA0183/RXP: now reaches J3.3 (Pin_3)
- net NMEA0183/RXN: now reaches J3.4 (Pin_4)
- net Microcontroller/AIS_UART_RX renamed Microcontroller/AIS_UART0_RX
- net Power/VP12V renamed VP12V
- net VP12V: now also J8.4 (Pin_4)
- new net Microcontroller/AIS_PPS: J5.4 (Pin_4)
- new net Microcontroller/AIS_UART1_RX: J5.5 (Pin_5)
- new net Microcontroller/AIS_UART1_TX: J5.3 (Pin_3)
- new net NMEA2000/CAN_H: J8.2 (Pin_2)
- new net NMEA2000/CAN_L: J8.5 (Pin_5)
- no-connect marks 29 -> 7
Other:
- added sheet NMEA0183 (nmea0183.kicad_sch)
- added sheet NMEA2000 (nmea2000.kicad_sch)
- sheet Microcontroller ports: added AIS_PPS, AIS_UART0_RX, AIS_UART1_RX, AIS_UART1_TX, CAN_RX, CAN_TX, MODEM_DTR, MODEM_PWR, MODEM_RX, MODEM_TX, NMEA0183_RX, NMEA0183_TX; removed AIS_UART_RX
- note added: "1 = GND 2 = CAN-H 3 = NC 4 = 12V 5 = CAN-L"
- note added: "Expirimental 2x3pin cable for external GPS (PPS)"
- note added: "TODO: - GPS ANTENNA MATCHING CIRCUIT - M12 CONNECTOR - SCHEMATIC CHECK - TEST POINTS - MOUNTING HOLES"
- note removed: "ADD filtering to GPS"
- note removed: "Fred?"
- note removed: "TODO: - POWER LEDs - USER LEDs - GPS ANTENNA MATCHING CIRCUIT - CAN DRIVER - NMEA 0183 - NMEA 2000 - M12 CONNECTOR - SCHEMATIC CHECK - TEST POINTS - MOUNTING HOLES - ??"
- note removed: "reverse polarity protection P fet and zener"
- moved on the sheet: R51, R52

Commit message: Clean up and testpoints
Parts:
- added H1, H2, H3, H4: MountingHole_Pad, MountingHole:MountingHole_3.2mm_M3_DIN965_Pad, symbol Mechanical:MountingHole_Pad
- added PoE+, PoE-, TP1, TP10, TP11, TP12, TP13, TP14, TP15, TP16, TP17, TP18, TP19, TP2, TP20, TP21, TP3, TP4, TP5, TP6, TP7, TP8, TP9: TestPoint, TestPoint:TestPoint_Pad_D1.5mm, symbol Connector:TestPoint
Connections:
- net Ethernet PHY/MDC: now also TP1.1
- net Ethernet PHY/MDIO: now also TP2.1
- net GND: now also H1.1, H2.1, H3.1, H4.1
- net Microcontroller/AIS_UART0_RX: now also TP19.1
- net Microcontroller/AIS_UART0_TX: now also TP18.1
- net Microcontroller/CAN_RX: now also TP20.1
- net Microcontroller/CAN_TX: now also TP21.1
- net Microcontroller/CH_DTR: now also TP16.1
- net Microcontroller/CH_RTS: now also TP17.1
- net Microcontroller/ESP_RXD0: now also TP14.1
- net Microcontroller/ESP_TXD0: now also TP15.1
- net Microcontroller/MODEM_DTR: now also TP6.1
- net Microcontroller/MODEM_PWR: now also TP5.1
- net Microcontroller/MODEM_RX: now also TP8.1
- net Microcontroller/MODEM_TX: now also TP7.1
- net Microcontroller/NMEA0183_RX: now also TP4.1
- net Microcontroller/NMEA0183_TX: now also TP3.1
- net Power/VN_PoE: now also PoE-.1
- net Power/VP_PoE: now also PoE+.1
- net Power/VP_USB: now also TP13.1
- net VDDA_3V3: now also TP12.1
- net VP12V: now also TP9.1
- net VP3V3: now also TP10.1
- net VP5V: now also TP11.1
Other:
- note added: "Experimental 2x3pin cable for external GPS (PPS)"
- note added: "TODO: - SCHEMATIC CHECK"
- note removed: "Expirimental 2x3pin cable for external GPS (PPS)"
- note removed: "TODO: - GPS ANTENNA MATCHING CIRCUIT - M12 CONNECTOR - SCHEMATIC CHECK - TEST POINTS - MOUNTING HOLES"

Commit message: Layout save
Parts:
- added D14, D15: D, Diode_SMD:D_1206_3216Metric, symbol Device:D
- renumbered PoE+ to PoE+1, PoE- to PoE-1
Connections:
- net VP12V: now also D14.1 (K), D15.1 (K); no longer J1.1 (Pin_1), J8.4 (Pin_4)
- new net: D14.2 (A), J1.1 (Pin_1)
- new net: D15.2 (A), J8.4 (Pin_4)
Other:
- note added: "TODO: - REVIEW SCHEMA - NMEA2000 only as INPUT"
- note removed: "TODO: - SCHEMATIC CHECK"

Commit message: Power layout started
Connections:
- net Ethernet PHY/MDC: no longer TP1.1
- net Ethernet PHY/MDIO: no longer TP2.1
- net Microcontroller/AIS_UART0_RX: no longer TP19.1
- net Microcontroller/AIS_UART0_TX: no longer TP18.1
- net Microcontroller/CAN_RX: no longer TP20.1
- net Microcontroller/CAN_TX: no longer TP21.1
- net Microcontroller/CH_DTR: no longer TP16.1
- net Microcontroller/CH_RTS: no longer TP17.1
- net Microcontroller/ESP_RXD0: no longer TP14.1
- net Microcontroller/ESP_TXD0: no longer TP15.1
- net Microcontroller/MODEM_DTR: no longer TP6.1
- net Microcontroller/MODEM_PWR: no longer TP5.1
- net Microcontroller/MODEM_RX: no longer TP8.1
- net Microcontroller/MODEM_TX: no longer TP7.1
- net Microcontroller/NMEA0183_RX: no longer TP4.1
- net Microcontroller/NMEA0183_TX: no longer TP3.1
- net NMEA0183/RXN: now also J3.3 (Pin_3); no longer J3.4 (Pin_4)
- net NMEA0183/RXP: now also J3.4 (Pin_4); no longer J3.3 (Pin_3)
- net NMEA0183/TXN: now also J3.1 (Pin_1); no longer J3.2 (Pin_2)
- net NMEA0183/TXP: now also J3.2 (Pin_2); no longer J3.1 (Pin_1)
- net Power/VN_PoE: no longer PoE-1.1
- net Power/VP_PoE: no longer PoE+1.1
- net Power/VP_USB: no longer TP13.1
- net VP12V: no longer TP9.1
- net VP3V3: no longer TP10.1
- net VP5V: no longer TP11.1
