File: ethernet.kicad_sch (KiCad schematic)
At the start: 1 part, among them U2 LAN8720A

Commit message: progress save
Parts:
- removed U2: LAN8720A, Package_DFN_QFN:VQFN-24-1EP_4x4mm_P0.5mm_EP2.5x2.5mm_ThermalVias, symbol Interface_Ethernet:LAN8720A
Changed lines of the file:
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@@
 	(generator_version "10.0")
 	(paper "A4")
-	(symbol
-		(lib_id "Interface_Ethernet:LAN8720A")
-		(at 152.4 91.44 0)
-		(unit 1)
-		(body_style 1)
-		(exclude_from_sim no)
-		(in_bom yes)
-		(on_board yes)
-		(in_pos_files yes)
-		(dnp no)
-		(fields_autoplaced yes)
-		(property "Reference" "U2"
-			(at 154.5433 119.38 0)
-			(show_name no)
-			(do_not_autoplace no)
-			(effects
-				(font
-					(size 1.27 1.27)
-				)
-				(justify left)
-			)
-		)
-		(property "Value" "LAN8720A"
-			(at 154.5433 121.92 0)
-			(show_name no)
-			(do_not_autoplace no)
-			(effects
-				(font
-					(size 1.27 1.27)
-				)
-				(justify left)
-			)
-		)
-		(property "Footprint" "Package_DFN_QFN:VQFN-24-1EP_4x4mm_P0.5mm_EP2.5x2.5mm_ThermalVias"
-			(at 153.67 118.11 0)
-			(hide yes)
-			(show_name no)
-			(do_not_autoplace no)
-			(effects
-				(font
-					(size 1.27 1.27)
-				)
-				(justify left)
-			)
-		)
-		(property "Datasheet" "http://ww1.microchip.com/downloads/en/DeviceDoc/8720a.pdf"
-			(at 147.32 115.57 0)
-			(hide yes)
-			(show_name no)
-			(do_not_autoplace no)
-			(effects
-				(font
-					(size 1.27 1.27)
-				)
-			)
-		)
-		(property "Description" "LAN8720 Ethernet PHY with RMII interface, QFN-24"
-			(at 152.4 91.44 0)
-			(hide yes)
-			(show_name no)
-			(do_not_autoplace no)
-			(effects
-				(font
-					(size 1.27 1.27)
-				)
-			)
-		)
-		(pin "16"
-		)
-		(pin "25"
-		)
-		(pin "2"
-		)
-		(pin "8"
-		)
-		(pin "17"
-		)
-		(pin "12"
-		)
-		(pin "19"
-		)
-		(pin "5"
-		)
-		(pin "4"
-		)
-		(pin "13"
-		)
-		(pin "1"
-		)
-		(pin "9"
-		)
-		(pin "11"
-		)
-		(pin "14"
-		)
-		(pin "23"
-		)
-		(pin "7"
-		)
-		(pin "15"
-		)
-		(pin "10"
-		)
-		(pin "3"
-		)
-		(pin "20"
-		)
-		(pin "6"
-		)
-		(pin "18"
-		)
-		(pin "22"
-		)
-		(pin "24"
-		)
-		(pin "21"
-		)
-		(instances
-			(project "AIS-Converter"
-				(path "/af2e2bda-c8b0-494b-9cbc-4303d4ae7608/80bdb5d0-cde6-4aa9-86eb-9bd054667ca4"
-					(reference "U2")
-					(unit 1)
-				)
-			)
-		)
-	)
 )
