File: ethernet.kicad_sch (KiCad schematic)
At the start: 0 parts

Commit message: Adding ethernet module and more
Parts:
- added C10, C11, C12, C9: 10pF, Capacitor_SMD:C_0402_1005Metric, symbol Device:C
- added C13: 470pF, Capacitor_SMD:C_0603_1608Metric, symbol Device:C
- added C14: 1uF, Capacitor_SMD:C_0603_1608Metric, symbol Device:C
- added D2: ESDS304, Package_TO_SOT_SMD:SOT-23-5, symbol Power_Protection:ESDS304
- added FB9: FerriteBead, symbol Device:FerriteBead
- added R10, R11, R12, R9: 49R9, Resistor_SMD:R_0402_1005Metric, symbol Device:R
- added U5: LAN8720A, Package_DFN_QFN:VQFN-24-1EP_4x4mm_P0.5mm_EP2.5x2.5mm_ThermalVias, symbol Rick:LAN8720A
Connections:
- new net: R10.1, R11.1, R12.1, R9.1
- new net: C13.1, C14.1, U5.6 (VDDCR)
- new net: FB9.2, U5.1 (VDD2A), U5.19 (VDD1A)
- new net: FB9.1, U5.9 (VDDIO)
- new net GND: C10.2, C11.2, C12.2, C13.2, C14.2, C9.2
- new net RXN: C12.1, U5.22 (RXN)
- new net RXP: C11.1, U5.23 (RXP)
- new net TXN: C10.1, U5.20 (TXN)
- new net TXP: C9.1, U5.21 (TXP)
Other:
- note added: "TVS 0402 between diff pairs eth GG0402052R542P"
- note added: "https://github.com/c-/ESP32-Ethgate/blob/main/ESP32-Ethgate.pdf https://github.com/Zelmoghazy/esp32-ethernet-lan8720 https://www.microchip.com/en-us/product/lan8720a https://ww1.microchip.com/downloads/aemDocuments/documents/OTH/ApplicationNotes/ApplicationNotes/00002157B.pdf https://www.olimex.com/Products/IoT/ESP32/ESP32-POE/open-source-hardware"
- note added: "https://ww1.microchip.com/downloads/en/DeviceDoc/evb8720sch.pdf"

Commit message: Ethernet progress, 40pin connector, save progress
Parts:
- added C15: 100nf, Capacitor_SMD:C_0603_1608Metric, symbol Device:C
- added C16, C17, C33: 100nF, Capacitor_SMD:C_0603_1608Metric, symbol Device:C
- added C18: 4u7F, Capacitor_SMD:C_0603_1608Metric, symbol Device:C
- added C32: 10n, Capacitor_SMD:C_0603_1608Metric, symbol Device:C
- added R34: 12k1, Resistor_SMD:R_0201_0603Metric, symbol Device:R
- added R37: 10k, Resistor_SMD:R_0603_1608Metric, symbol Device:R
- added R38: 1k5, Resistor_SMD:R_0603_1608Metric, symbol Device:R
- added R39: 33R, Resistor_SMD:R_0603_1608Metric, symbol Device:R
- added R40, R41, R42: 10R, Resistor_SMD:R_0603_1608Metric, symbol Device:R
- added R43, R44, R45, R46, R47, R48, R49, R50: 1k5, symbol Device:R
- FB9: value FerriteBead -> 2A/0.050 DCR; footprint (none) -> Inductor_SMD:C_0603_1608Metric
Connections:
- net ETH_ACT_LED: now also U5.3 (LED1/REGOFF)
- net ETH_LINK_LED: now also U5.2 (LED2/~{INTSEL})
- net GND: now also D2.2 (A), U5.25 (GND), C15.2, C16.2, C17.2, C18.2, C32.2, C33.2, R34.2, R47.2, R48.2, R49.2, R50.2
- net RXN: now also D2.5 (K), R12.2
- net RXP: now also D2.4 (K), R11.2
- net TXN: now also D2.3 (K), R10.2
- net TXP: now also D2.1 (K), R9.2
- net VP3V3: now reaches R10.1, R11.1, R12.1, R9.1
- net VP3V3: now also FB9.1, U5.9 (VDDIO), C15.1, R37.1, R38.1, R43.1, R44.1, R45.1, R46.1
- net at C13.1, C14.1, U5.6 (VDDCR): now also C32.1
- net VP3V3_VDDA: now reaches FB9.2, U5.1 (VDD2A), U5.19 (VDD1A)
- net VP3V3_VDDA: now also C16.1, C17.1, C18.1
- net RXER/PHYADD0: now reaches U5.10 (RXER/PHYAD0)
- net RXER/PHYADD0: now also R46.2, R47.1
- net at U5.11 (CRS_DV/MODE2): now also R42.1
- net MDIO: now reaches U5.12 (MDIO)
- net MDIO: now also R38.2
- net MDC: now reaches U5.13 (MDC)
- net at U5.15 (~{RST}): now also C33.1, R37.2
- net TXEN: now reaches U5.16 (TXEN)
- net TXD0: now reaches U5.17 (TXD0)
- net TXD1: now reaches U5.18 (TXD1)
- net at U5.24 (RBIAS): now also R34.1
- net at U5.5 (XTAL1/CLKIN): now also R39.2
- net at U5.7 (RXD1/MODE1): now also R41.1
- net at U5.8 (RXD0/MODE0): now also R40.1
- new net CRS_DV/MODE2: R42.2, R45.2, R48.1
- new net ETH_CLK: R39.1
- new net RXD0/MODE0: R40.2, R44.2, R50.1
- new net RXD1/MODE1: R41.2, R43.2, R49.1
- no-connect marks 0 -> 2
Other:
- note added: "Add strap on resitors for regoff and intsel here for readability"
- note added: "PHYAD[0] = 0 (RXER pull-down) MODE[2:0] = 111 (All capable, AUTO MDI-X ON)"
- note added: "REGOFF = 1 (1V2 ON) ~{INTSEL} = 1 (External Clock)"
- note added: "diff pair 100ohm Z"
- note added: "single ended 50ohm Z"
- note removed: "https://github.com/c-/ESP32-Ethgate/blob/main/ESP32-Ethgate.pdf https://github.com/Zelmoghazy/esp32-ethernet-lan8720 https://www.microchip.com/en-us/product/lan8720a https://ww1.microchip.com/downloads/aemDocuments/documents/OTH/ApplicationNotes/ApplicationNotes/00002157B.pdf https://www.olimex.com/Products/IoT/ESP32/ESP32-POE/open-source-hardware"
- note removed: "https://ww1.microchip.com/downloads/en/DeviceDoc/evb8720sch.pdf"
- moved on the sheet: C10, C11, C12, C13, C14, C9, D2, FB9, R10, R11, R12, R9

Commit message: Layout save
Parts:
- FB9: footprint Inductor_SMD:C_0603_1608Metric -> Inductor_SMD:L_0603_1608Metric
- R34: footprint Resistor_SMD:R_0201_0603Metric -> Resistor_SMD:R_0402_1005Metric
- R40, R41, R42: footprint Resistor_SMD:R_0603_1608Metric -> Resistor_SMD:R_0402_1005Metric
- R43, R44, R45, R46, R47, R48, R49, R50: footprint (none) -> Resistor_SMD:R_0603_1608Metric
Changed lines of the file:
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@@
 			)
 		)
-		(property "Footprint" ""
+		(property "Footprint" "Resistor_SMD:R_0603_1608Metric"
 			(at 366.522 127 90)
 			(hide yes)
@@
 			)
 		)
-		(property "Footprint" ""
+		(property "Footprint" "Resistor_SMD:R_0603_1608Metric"
 			(at 360.172 175.26 90)
 			(hide yes)
@@
 			)
 		)
-		(property "Footprint" "Resistor_SMD:R_0201_0603Metric"
+		(property "Footprint" "Resistor_SMD:R_0402_1005Metric"
 			(at 259.842 179.07 90)
 			(hide yes)
@@
 			)
 		)
-		(property "Footprint" ""
+		(property "Footprint" "Resistor_SMD:R_0603_1608Metric"
 			(at 374.142 120.65 90)
 			(hide yes)
@@
 			)
 		)
-		(property "Footprint" "Resistor_SMD:R_0603_1608Metric"
+		(property "Footprint" "Resistor_SMD:R_0402_1005Metric"
 			(at 354.33 150.368 90)
 			(hide yes)
@@
 			)
 		)
-		(property "Footprint" ""
+		(property "Footprint" "Resistor_SMD:R_0603_1608Metric"
 			(at 375.412 175.26 90)
 			(hide yes)
@@
 			)
 		)
-		(property "Footprint" ""
+		(property "Footprint" "Resistor_SMD:R_0603_1608Metric"
 			(at 358.902 120.65 90)
 			(hide yes)
@@
 			)
 		)
-		(property "Footprint" ""
+		(property "Footprint" "Resistor_SMD:R_0603_1608Metric"
 			(at 381.762 127 90)
 			(hide yes)
@@
 			)
 		)
-		(property "Footprint" "Inductor_SMD:C_0603_1608Metric"
+		(property "Footprint" "Inductor_SMD:L_0603_1608Metric"
 			(at 234.95 109.728 90)
 			(hide yes)
@@
 			)
 		)
-		(property "Footprint" "Resistor_SMD:R_0603_1608Metric"
+		(property "Footprint" "Resistor_SMD:R_0402_1005Metric"
 			(at 344.17 152.908 90)
 			(hide yes)
@@
 			)
 		)
-		(property "Footprint" ""
+		(property "Footprint" "Resistor_SMD:R_0603_1608Metric"
 			(at 367.792 175.26 90)
 			(hide yes)
@@
 			)
 		)
-		(property "Footprint" ""
+		(property "Footprint" "Resistor_SMD:R_0603_1608Metric"
 			(at 383.032 175.26 90)
 			(hide yes)
@@
 			)
 		)
-		(property "Footprint" "Resistor_SMD:R_0603_1608Metric"
+		(property "Footprint" "Resistor_SMD:R_0402_1005Metric"
 			(at 335.28 157.988 90)
 			(hide yes)
