File: modem.kicad_sch (KiCad schematic)
At the start: 44 parts, among them Q1 MMBT3904, Q2 MMBT3904, Q3 MMBT3904, Q4 MMBT3904, U7 SMN-304, U8 SIM7080G

Commit message: progress save
Parts:
- added U3: New Version, Rick:dAISy-catcher-11mm, symbol Rick:dAISy-catcher
- U7: footprint 1_Custom_Rick:SMN-304 -> Rick:SMN-304
- U8: footprint 1_Custom_Rick:XCVR_SIM7080G -> Rick:XCVR_SIM7080G
Changed lines of the file:
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@@
 			)
 		)
-		(property "Footprint" "1_Custom_Rick:XCVR_SIM7080G"
+		(property "Footprint" "Rick:XCVR_SIM7080G"
 			(at 196.85 153.67 0)
 			(hide yes)
@@
 			)
 		)
-		(property "Footprint" "1_Custom_Rick:SMN-304"
+		(property "Footprint" "Rick:SMN-304"
 			(at 99.822 153.67 0)
 			(hide yes)
@@
 					(unit 1)
 				)
+			)
+		)
+	)
+	(symbol
+		(lib_id "Rick:dAISy-catcher")
+		(at 85.09 181.61 0)
+		(unit 1)
+		(body_style 1)
+		(exclude_from_sim no)
+		(in_bom yes)
+		(on_board yes)
+		(in_pos_files yes)
+		(dnp no)
+		(fields_autoplaced yes)
+		(property "Reference" "U3"
+			(at 93.98 180.3399 0)
+			(show_name no)
+			(do_not_autoplace no)
+			(effects
+				(font
+					(size 1.27 1.27)
+				)
+				(justify left)
+			)
+		)
+		(property "Value" "New Version"
+			(at 93.98 182.8799 0)
+			(show_name no)
+			(do_not_autoplace no)
+			(effects
+				(font
+					(size 1.27 1.27)
+				)
+				(justify left)
+			)
+		)
+		(property "Footprint" "Rick:dAISy-catcher-11mm"
+			(at 85.09 181.61 0)
+			(hide yes)
+			(show_name no)
+			(do_not_autoplace no)
+			(effects
+				(font
+					(size 1.27 1.27)
+				)
+			)
+		)
+		(property "Datasheet" ""
+			(at 85.09 181.61 0)
+			(hide yes)
+			(show_name no)
+			(do_not_autoplace no)
+			(effects
+				(font
+					(size 1.27 1.27)
+				)
+			)
+		)
+		(property "Description" ""
+			(at 85.09 181.61 0)
+			(hide yes)
+			(show_name no)
+			(do_not_autoplace no)
+			(effects
+				(font
+					(size 1.27 1.27)
+				)
+			)
+		)
+		(instances
+			(project "AIS-Converter"
+				(path "/af2e2bda-c8b0-494b-9cbc-4303d4ae7608/35a6c23c-94a1-420f-9e5f-a39ff34ffec8"
+					(reference "U3")
+					(unit 1)
+				)
