File: power.kicad_sch (KiCad schematic)
At the start: 0 parts

Commit message: progress save
Parts:
- added U2: AG9905-LP, Rick:AG9905-LP, symbol Rick:AG9905-LP
Connections:
- new net: U2.1 (+VDC), U2.2 (+VDC)
- new net VIN+: U2.5 (VIN+), U2.6 (VIN+)
- new net VIN-: U2.7 (VIN-), U2.8 (VIN-)
Other:
- note added: "Ag9905-LP"
- note added: "Diode bridge in connector"
Changed lines of the file:
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@@
+		)
+	)
+	(text "Diode bridge in connector"
+		(exclude_from_sim no)
+		(at 58.674 99.314 0)
+		(effects
+			(font
+				(size 1.27 1.27)
+			)
+		)
+	)
+	(text "Ag9905-LP"
+		(exclude_from_sim no)
+		(at 80.518 59.182 0)
+		(effects
+			(font
+				(size 1.27 1.27)
+			)
 		)
 	)
@@
 		)
 	)
+	(symbol
+		(lib_id "Rick:AG9905-LP")
+		(at 86.36 100.33 0)
+		(unit 1)
+		(body_style 1)
+		(exclude_from_sim no)
+		(in_bom yes)
+		(on_board yes)
+		(in_pos_files yes)
+		(dnp no)
+		(fields_autoplaced yes)
+		(property "Reference" "U2"
+			(at 86.36 85.09 0)
+			(show_name no)
+			(do_not_autoplace no)
+			(effects
+				(font
+					(size 1.27 1.27)
+				)
+			)
+		)
+		(property "Value" "AG9905-LP"
+			(at 86.36 87.63 0)
+			(show_name no)
+			(do_not_autoplace no)
+			(effects
+				(font
+					(size 1.27 1.27)
+				)
+			)
+		)
+		(property "Footprint" "Rick:AG9905-LP"
+			(at 80.772 112.014 0)
+			(hide yes)
+			(show_name no)
+			(do_not_autoplace no)
+			(effects
+				(font
+					(size 1.27 1.27)
+				)
+			)
+		)
+		(property "Datasheet" ""
+			(at 86.36 100.33 0)
+			(hide yes)
+			(show_name no)
+			(do_not_autoplace no)
+			(effects
+				(font
+					(size 1.27 1.27)
+				)
+			)
+		)
+		(property "Description" ""
+			(at 86.36 100.33 0)
+			(hide yes)
+			(show_name no)
+			(do_not_autoplace no)
+			(effects
+				(font
+					(size 1.27 1.27)
+				)
+			)
+		)
+		(pin "6"
+		)
+		(pin "8"
+		)
+		(pin "3"
+		)
+		(pin "1"
+		)
+		(pin "5"
+		)
+		(pin "7"
+		)
+		(pin "2"
+		)
+		(pin "4"
+		)
+		(instances
+			(project "AIS-Converter"
+				(path "/af2e2bda-c8b0-494b-9cbc-4303d4ae7608/129c204b-2a58-4519-abe1-43b32e5912d0"
+					(reference "U2")
+					(unit 1)
+				)
+			)
+		)
+	)
