File: nmea0183.kicad_sch (KiCad schematic)
At the start: 6 parts, among them U15 MAX490E

Commit message: Layout save
Parts:
- R57, R58: footprint (none) -> Resistor_SMD:R_0603_1608Metric
Changed lines of the file:
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@@
 			)
 		)
-		(property "Footprint" ""
+		(property "Footprint" "Resistor_SMD:R_0603_1608Metric"
 			(at 170.942 133.35 90)
 			(hide yes)
@@
 			)
 		)
-		(property "Footprint" ""
+		(property "Footprint" "Resistor_SMD:R_0603_1608Metric"
 			(at 155.702 133.35 90)
 			(hide yes)
