File: AIS-Converter.kicad_pcb (KiCad board)
At the start: 4 copper layers, 135 x 56 mm, 59 parts, among them J1 Conn_01x02, J2 USB_C_Receptacle_USB2.0_16P, J3 Conn_01x04, J4 Raspberry_Pi_4, J6 Conn_Coaxial_Small, J7 Conn_Coaxial_Small, Q1 MMBT3904, Q2 MMBT3904, Q3 MMBT3904, Q4 MMBT3904, U1 ESP32-WROOM-32E, U2 AG9905-LP, U3 dAISy-catcher, U4 HY931147C, U5 LAN8720A, U7 SMN-304, U8 SIM7080G

Commit message: Layout save
Parts:
- added C1: C, Capacitor_SMD:C_0603_1608Metric, F.Cu at (45.5, 107.2)
- added C10: 10pF, Capacitor_SMD:C_0402_1005Metric, F.Cu at (258.9, 81.7)
- added C11: 10pF, Capacitor_SMD:C_0402_1005Metric, F.Cu at (258.9, 83.7)
- added C12: 10pF, Capacitor_SMD:C_0402_1005Metric, F.Cu at (258.9, 85.7)
- added C13: 470pF, Capacitor_SMD:C_0603_1608Metric, F.Cu at (264.9, 94.4)
- added C14: 1uF, Capacitor_SMD:C_0603_1608Metric, F.Cu at (264.9, 96.9)
- added C15: 100nf, Capacitor_SMD:C_0603_1608Metric, F.Cu at (264.9, 99.4)
- added C16: 100nF, Capacitor_SMD:C_0603_1608Metric, F.Cu at (264.9, 101.9)
- added C17: 100nF, Capacitor_SMD:C_0603_1608Metric, F.Cu at (264.9, 104.4)
- added C18: 4u7F, Capacitor_SMD:C_0603_1608Metric, F.Cu at (264.9, 106.9)
- added C19: 22n, Capacitor_SMD:C_0603_1608Metric, F.Cu at (417.3, -34.0)
- added C2: C_Polarized, Capacitor_SMD:C_0603_1608Metric, F.Cu at (45.5, 109.7)
- added C3: C, Capacitor_SMD:C_0603_1608Metric, F.Cu at (45.5, 112.2)
- added C32: 10n, Capacitor_SMD:C_0603_1608Metric, F.Cu at (264.9, 109.5)
- added C33: 100nF, Capacitor_SMD:C_0603_1608Metric, F.Cu at (264.9, 112.0)
- added C34: 100nF, Capacitor_SMD:C_0603_1608Metric, F.Cu at (328.2, 107.5)
- added C35: 100nF, Capacitor_SMD:C_0603_1608Metric, F.Cu at (306.8, 108.0)
- added C38: 100pF, Capacitor_SMD:C_0603_1608Metric, F.Cu at (100.9, 84.4)
- added C4: 100n, Capacitor_SMD:C_0603_1608Metric, F.Cu at (98.4, 77.8)
- added C5: 100n, Capacitor_SMD:C_0603_1608Metric, F.Cu at (90.0, 56.3)
- added C6: 100n, Capacitor_SMD:C_0603_1608Metric, F.Cu at (90.0, 58.8)
- added C7: 10uF, Capacitor_SMD:C_0603_1608Metric, F.Cu at (45.5, 114.8)
- added C8: 4u7F, Capacitor_SMD:C_0603_1608Metric, F.Cu at (45.5, 117.3)
- added C9: 10pF, Capacitor_SMD:C_0402_1005Metric, F.Cu at (258.9, 79.7)
- added D1: SMAJ58A, Diode_SMD:D_SMA, F.Cu at (248.5, 101.5)
- added D10: PWR_3V3, LED_SMD:LED_0603_1608Metric, F.Cu at (67.6, 103.8)
- added D11: SM712_SOT23, Package_TO_SOT_SMD:SOT-23, F.Cu at (323.7, 108.4)
- added D12: SM712_SOT23, Package_TO_SOT_SMD:SOT-23, F.Cu at (323.7, 112.9)
- added D13: SM24CANB-02HTG, Package_TO_SOT_SMD:SOT-23, F.Cu at (311.2, 108.9)
- added D2: ESDS304, Package_TO_SOT_SMD:SOT-23-5, F.Cu at (277.5, 103.5)
- added D3: 0R, Diode_SMD:D_0603_1608Metric, F.Cu at (67.6, 98.7)
- added D4: PWR_5V, LED_SMD:LED_0603_1608Metric, F.Cu at (67.6, 101.3)
- added FB1: 0R, Inductor_SMD:L_0603_1608Metric, F.Cu at (245.5, 98.0)
- added FB2: 0R, Inductor_SMD:L_0603_1608Metric, F.Cu at (247.0, 96.5)
- added FB3: 0R, Inductor_SMD:L_0603_1608Metric, F.Cu at (245.5, 94.8)
- added FB4: 0R, Inductor_SMD:L_0603_1608Metric, F.Cu at (251.5, 98.0)
- added FB5: 0R, Inductor_SMD:L_0603_1608Metric, F.Cu at (250.0, 96.5)
- added FB6: 0R, Inductor_SMD:L_0603_1608Metric, F.Cu at (251.5, 95.0)
- added FB7: 0R, Inductor_SMD:L_0603_1608Metric, F.Cu at (49.5, 119.8)
- added FB8: 0R, Inductor_SMD:L_0603_1608Metric, F.Cu at (90.0, 61.3)
- added FB9: 2A/0.050 DCR, Inductor_SMD:L_0603_1608Metric, F.Cu at (268.9, 94.4)
- added H1: MountingHole_Pad, MountingHole:MountingHole_3.2mm_M3_DIN965_Pad, F.Cu at (120.2, 55.5)
- added H2: MountingHole_Pad, MountingHole:MountingHole_3.2mm_M3_DIN965_Pad, F.Cu at (241.8, 55.5)
- added H3: MountingHole_Pad, MountingHole:MountingHole_3.2mm_M3_DIN965_Pad, F.Cu at (120.2, 113.5)
- added H4: MountingHole_Pad, MountingHole:MountingHole_3.2mm_M3_DIN965_Pad, F.Cu at (241.7, 113.5)
- added J5: Conn_01x02, Connector_PinSocket_2.54mm:PinSocket_2x03_P2.54mm_Vertical, F.Cu at (80.6, 78.6)
- added J8: M12A-05PMMR-SF7003, Rick:M12A05PMMRSF7003, F.Cu at (212.0, 114.0)
- added L1: 68nH, Inductor_SMD:L_0603_1608Metric, F.Cu at (100.9, 86.9)
- added PoE+1: TestPoint, TestPoint:TestPoint_Pad_D1.5mm, B.Cu at (390.0, -59.6)
- added PoE-1: TestPoint, TestPoint:TestPoint_Pad_D1.5mm, B.Cu at (390.0, -56.0)
- added Q7: UMH3N, Package_TO_SOT_SMD:SOT-363_SC-70-6, F.Cu at (93.9, 56.8)
- added R10: 49R9, Resistor_SMD:R_0402_1005Metric, F.Cu at (261.9, 81.7)
- added R11: 49R9, Resistor_SMD:R_0402_1005Metric, F.Cu at (261.9, 83.7)
- added R12: 49R9, Resistor_SMD:R_0402_1005Metric, F.Cu at (261.9, 85.7)
- added R3: 0R, Resistor_SMD:R_0201_0603Metric, F.Cu at (70.9, 98.2)
- added R34: 12k1, Resistor_SMD:R_0201_0603Metric, F.Cu at (276.1, 106.6)
- added R35: 1k5, Resistor_SMD:R_0603_1608Metric, F.Cu at (417.3, -31.5)
- added R36: 1k5, Resistor_SMD:R_0603_1608Metric, F.Cu at (417.3, -29.0)
- added R37: 10k, Resistor_SMD:R_0603_1608Metric, F.Cu at (268.9, 96.9)
- added R38: 1k5, Resistor_SMD:R_0603_1608Metric, F.Cu at (268.9, 99.4)
- added R39: 33R, Resistor_SMD:R_0603_1608Metric, F.Cu at (268.9, 101.9)
- added R4: 0R, Resistor_SMD:R_0201_0603Metric, F.Cu at (97.6, 70.4)
- added R40: 10R, Resistor_SMD:R_0603_1608Metric, F.Cu at (268.9, 104.4)
- added R41: 10R, Resistor_SMD:R_0603_1608Metric, F.Cu at (268.9, 106.9)
- added R42: 10R, Resistor_SMD:R_0603_1608Metric, F.Cu at (268.9, 109.5)
- added R43: 1k5, Resistor_SMD:R_0603_1608Metric, F.Cu at (268.9, 112.0)
- added R44: 1k5, Resistor_SMD:R_0603_1608Metric, F.Cu at (272.9, 94.4)
- added R45: 1k5, Resistor_SMD:R_0603_1608Metric, F.Cu at (272.9, 96.9)
- added R46: 1k5, Resistor_SMD:R_0603_1608Metric, F.Cu at (272.9, 99.4)
- added R47: 1k5, Resistor_SMD:R_0603_1608Metric, F.Cu at (272.9, 101.9)
- added R48: 1k5, Resistor_SMD:R_0603_1608Metric, F.Cu at (272.9, 104.4)
- added R49: 1k5, Resistor_SMD:R_0603_1608Metric, F.Cu at (272.9, 106.9)
- added R5: 0R, Resistor_SMD:R_0201_0603Metric, F.Cu at (97.6, 72.2)
- added R50: 1k5, Resistor_SMD:R_0603_1608Metric, F.Cu at (272.9, 109.5)
- added R51: 0R, Resistor_SMD:R_0603_1608Metric, F.Cu at (73.8, 85.1)
- added R52: 0R, Resistor_SMD:R_0603_1608Metric, F.Cu at (73.8, 87.6)
- added R53: 1k5, Resistor_SMD:R_0603_1608Metric, F.Cu at (53.5, 107.2)
- added R54: 680R, Resistor_SMD:R_0603_1608Metric, F.Cu at (53.5, 109.7)
- added R55: 0R, Resistor_SMD:R_0603_1608Metric, F.Cu at (53.5, 112.2)
- added R56: 0R, Resistor_SMD:R_0603_1608Metric, F.Cu at (53.5, 114.8)
- added R57: 0R, Resistor_SMD:R_0603_1608Metric, F.Cu at (328.2, 110.0)
- added R58: 0R, Resistor_SMD:R_0603_1608Metric, F.Cu at (328.2, 112.5)
- added R59: 0R, Resistor_SMD:R_0603_1608Metric, F.Cu at (90.0, 66.3)
- added R6: 0R, Resistor_SMD:R_0201_0603Metric, F.Cu at (97.6, 73.9)
- added R60: 0R, Resistor_SMD:R_0603_1608Metric, F.Cu at (306.8, 110.5)
- added R61: 22R, Resistor_SMD:R_0603_1608Metric, F.Cu at (100.9, 89.4)
- added R7: 0R, Resistor_SMD:R_0201_0603Metric, F.Cu at (97.6, 75.7)
- added R8: 10k, Resistor_SMD:R_0603_1608Metric, F.Cu at (90.0, 63.8)
- added R9: 49R9, Resistor_SMD:R_0402_1005Metric, F.Cu at (261.9, 79.7)
- added TP1: TestPoint, TestPoint:TestPoint_Pad_D1.5mm, B.Cu at (390.0, -52.5)
- added TP10: TestPoint, TestPoint:TestPoint_Pad_D1.5mm, B.Cu at (37.4, 54.3)
- added TP11: TestPoint, TestPoint:TestPoint_Pad_D1.5mm, B.Cu at (41.0, 36.5)
- added TP12: TestPoint, TestPoint:TestPoint_Pad_D1.5mm, B.Cu at (397.1, -56.0)
- added TP13: TestPoint, TestPoint:TestPoint_Pad_D1.5mm, B.Cu at (41.0, 43.6)
- added TP14: TestPoint, TestPoint:TestPoint_Pad_D1.5mm, B.Cu at (41.0, 47.2)
- added TP15: TestPoint, TestPoint:TestPoint_Pad_D1.5mm, B.Cu at (41.0, 50.8)
- added TP16: TestPoint, TestPoint:TestPoint_Pad_D1.5mm, B.Cu at (41.0, 54.3)
- added TP17: TestPoint, TestPoint:TestPoint_Pad_D1.5mm, B.Cu at (44.5, 36.5)
- added TP18: TestPoint, TestPoint:TestPoint_Pad_D1.5mm, B.Cu at (44.5, 40.1)
- added TP19: TestPoint, TestPoint:TestPoint_Pad_D1.5mm, B.Cu at (52.0, 42.5)
- added TP2: TestPoint, TestPoint:TestPoint_Pad_D1.5mm, B.Cu at (390.0, -48.9)
- added TP20: TestPoint, TestPoint:TestPoint_Pad_D1.5mm, B.Cu at (44.5, 47.2)
- added TP21: TestPoint, TestPoint:TestPoint_Pad_D1.5mm, B.Cu at (44.5, 50.8)
- added TP22: TestPoint, TestPoint:TestPoint_Pad_D1.5mm, F.Cu at (62.5, 115.9)
- added TP23: TestPoint, TestPoint:TestPoint_Pad_D1.5mm, F.Cu at (62.5, 119.5)
- added TP24: TestPoint, TestPoint:TestPoint_Pad_D1.5mm, F.Cu at (62.5, 123.0)
- added TP3: TestPoint, TestPoint:TestPoint_Pad_D1.5mm, B.Cu at (33.9, 50.8)
- added TP4: TestPoint, TestPoint:TestPoint_Pad_D1.5mm, B.Cu at (33.9, 54.3)
- added TP5: TestPoint, TestPoint:TestPoint_Pad_D1.5mm, B.Cu at (37.4, 36.5)
- added TP6: TestPoint, TestPoint:TestPoint_Pad_D1.5mm, B.Cu at (37.4, 40.1)
- added TP7: TestPoint, TestPoint:TestPoint_Pad_D1.5mm, B.Cu at (37.4, 43.6)
- added TP8: TestPoint, TestPoint:TestPoint_Pad_D1.5mm, B.Cu at (37.4, 47.2)
- added TP9: TestPoint, TestPoint:TestPoint_Pad_D1.5mm, B.Cu at (37.4, 50.8)
- added U10: MAX40200AUK, Package_TO_SOT_SMD:SOT-23-5, F.Cu at (58.1, 117.6)
- added U11: B1205S-2WR3, Rick:B1205S-2WR3, F.Cu at (55.0, 101.7)
- added U12: CH340C, Package_SO:SOIC-16_3.9x9.9mm_P1.27mm, F.Cu at (92.2, 75.5)
- added U13: USBLC6-2SC6, Package_TO_SOT_SMD:SOT-23-6, F.Cu at (78.3, 88.4)
- added U14: NCP1117-3.3_TO252, Package_TO_SOT_SMD:TO-252-2, F.Cu at (67.6, 110.1)
- added U15: MAX490E, Package_SO:SOIC-8_3.9x4.9mm_P1.27mm, F.Cu at (325.5, 103.0)
- added U16: TJA1051T-3, Package_SO:SOIC-8_3.9x4.9mm_P1.27mm, F.Cu at (309.0, 103.5)
- added U6: MAX40200AUK, Package_TO_SOT_SMD:SOT-23-5, F.Cu at (58.1, 108.4)
- added U9: MAX40200AUK, Package_TO_SOT_SMD:SOT-23-5, F.Cu at (58.1, 113.0)
- J3: value Conn_01x04 -> Conn_01x05; footprint Rick:J_Wurth_WR-TBL_691322110004 -> Rick:J_Wurth_WR-TBL_691322110005
- J4: value Raspberry_Pi_4 -> Raspberry_Pi_40pin_Connector
- moved G*** 106.0 mm to (160.5, 271.0)
- moved U5 61.8 mm to (249.8, 78.1)
- moved U2 50.3 mm to (206.2, 95.2)
- moved J3 41.8 mm to (172.0, 116.0)
- moved U4 39.6 mm to (230.0, 113.4)
- moved J2 38.5 mm to (129.5, 122.0)
- moved U7 31.5 mm to (162.0, 117.0)
- moved U1 24.2 mm to (207.8, 58.1)
- moved J4 13.6 mm to (132.9, 61.3)
- moved FF 13.6 mm to (128.0, 109.0)
- moved U3 13.6 mm to (128.0, 109.0)
- moved J1 11.8 mm to (192.0, 116.0)
- moved J6 3.00 mm to (151.0, 119.5)
- moved J7 2.00 mm to (140.0, 119.5)
Connections:
- net Net-(J2-D+-PadA6) renamed /DP
- net Net-(J2-D--PadA7) renamed /DN
- net Net-(J4-5V-Pad2) renamed VP5V
- C23 pad 1: VBAT -> VP3V3
- C26 pad 1: VBAT -> VP3V3
- C27 pad 1: VBAT -> VP3V3
- C28 pad 1: VBAT -> VP3V3
- C29 pad 1: VBAT -> VP3V3
- C31 pad 1: /Modem/SIM_ANT -> /ANT
- D5 pad 1: VBAT -> VP3V3
- J1 pad 1: unconnected-(J1-Pin_1-Pad1) -> VP12V
- J1 pad 2: unconnected-(J1-Pin_2-Pad2) -> GND
- J3 pad 1: unconnected-(J3-Pin_1-Pad1) -> /NMEA0183/TXP
- J3 pad 2: unconnected-(J3-Pin_2-Pad2) -> /NMEA0183/TXN
- J3 pad 3: unconnected-(J3-Pin_3-Pad3) -> /NMEA0183/RXP
- J3 pad 4: unconnected-(J3-Pin_4-Pad4) -> /NMEA0183/RXN
- J4 pad 1: Net-(J4-3V3-Pad1) -> unconnected-(J4-3V3-Pad1)
- J4 pad 10: unconnected-(J4-GPIO15/UART_RXD-Pad10) -> Net-(J4-GPIO15/UART_RXD)
- J4 pad 14: Net-(J4-GND-Pad14) -> GND
- J4 pad 17: Net-(J4-3V3-Pad1) -> unconnected-(J4-3V3-Pad1)_1
- J4 pad 20: Net-(J4-GND-Pad14) -> GND
- J4 pad 25: Net-(J4-GND-Pad14) -> GND
- J4 pad 30: Net-(J4-GND-Pad14) -> GND
- J4 pad 34: Net-(J4-GND-Pad14) -> GND
- J4 pad 39: Net-(J4-GND-Pad14) -> GND
- J4 pad 6: Net-(J4-GND-Pad14) -> GND
- J4 pad 8: unconnected-(J4-GPIO14/UART_TXD-Pad8) -> Net-(J4-GPIO14/UART_TXD)
- J4 pad 9: Net-(J4-GND-Pad14) -> GND
- J6 pad 5: /Modem/SIM_ANT -> /ANT
- J7 pad 5: /Modem/GNSS_ANT -> /ANT
- Q1 pad 2: /Modem/DTR -> /Microcontroller/MODEM_DTR
- Q2 pad 3: /Modem/TXD -> /Microcontroller/MODEM_TX
- Q3 pad 2: /Modem/RXD -> /Microcontroller/MODEM_RX
- R17 pad 1: /Modem/DTR -> /Microcontroller/MODEM_DTR
- R17 pad 2: VBAT -> VP3V3
- R18 pad 1: VBAT -> VP3V3
- R18 pad 2: /Modem/TXD -> /Microcontroller/MODEM_TX
- R20 pad 1: /Modem/RXD -> /Microcontroller/MODEM_RX
- R20 pad 2: VBAT -> VP3V3
- R22 pad 1: /Modem/PWR_KEY -> /Microcontroller/MODEM_PWR
- R31 pad 2: /Modem/SIM_ANT -> /ANT
- R33 pad 1: VBAT -> VP3V3
- U1 pad 10: unconnected-(U1-IO25-Pad10) -> /Ethernet PHY/RXD0/MODE0
- U1 pad 11: unconnected-(U1-IO26-Pad11) -> /Ethernet PHY/RXD1/MODE1
- U1 pad 12: unconnected-(U1-IO27-Pad12) -> /Ethernet PHY/CRS_DV/MODE2
- U1 pad 13: unconnected-(U1-IO14-Pad13) -> /Microcontroller/AIS_UART0_RX
- U1 pad 14: unconnected-(U1-IO12-Pad14) -> Net-(U1-IO12)
- U1 pad 16: unconnected-(U1-IO13-Pad16) -> /Microcontroller/AIS_UART0_TX
- U1 pad 2: unconnected-(U1-VDD-Pad2) -> Net-(U1-VDD)
- U1 pad 25: unconnected-(U1-IO0-Pad25) -> Net-(Q7B-C2)
- U1 pad 26: unconnected-(U1-IO4-Pad26) -> /Microcontroller/MODEM_RX
- U1 pad 27: unconnected-(U1-IO16-Pad27) -> /Microcontroller/MODEM_TX
- U1 pad 28: unconnected-(U1-IO17-Pad28) -> /Ethernet PHY/ETH_CLK
- U1 pad 3: unconnected-(U1-EN-Pad3) -> Net-(Q7A-C1)
- U1 pad 30: unconnected-(U1-IO18-Pad30) -> /Ethernet PHY/MDIO
- U1 pad 31: unconnected-(U1-IO19-Pad31) -> /Ethernet PHY/TXD0
- U1 pad 33: unconnected-(U1-IO21-Pad33) -> /Ethernet PHY/TXEN
- U1 pad 34: unconnected-(U1-RXD0/IO3-Pad34) -> /Microcontroller/ESP_RXD0
- U1 pad 35: unconnected-(U1-TXD0/IO1-Pad35) -> /Microcontroller/ESP_TXD0
- U1 pad 36: unconnected-(U1-IO22-Pad36) -> /Ethernet PHY/TXD1
- U1 pad 37: unconnected-(U1-IO23-Pad37) -> /Ethernet PHY/MDC
- U1 pad 4: unconnected-(U1-SENSOR_VP-Pad4) -> /Microcontroller/MODEM_DTR
- U1 pad 6: unconnected-(U1-IO34-Pad6) -> /Microcontroller/CAN_TX
- U1 pad 7: unconnected-(U1-IO35-Pad7) -> /Microcontroller/CAN_RX
- U1 pad 8: unconnected-(U1-IO32-Pad8) -> /Microcontroller/NMEA0183_TX
- U1 pad 9: unconnected-(U1-IO33-Pad9) -> /Microcontroller/NMEA0183_RX
- U2 pad 3: unconnected-(U2--VDC-Pad3) -> Net-(U2--VDC)
- U2 pad 4: unconnected-(U2-ADJ-Pad4) -> Net-(U2-ADJ)
- U4 pad G+: unconnected-(U4-PadG+) -> /VDDA_3V3
- U4 pad G-: unconnected-(U4-PadG-) -> Net-(R36-Pad1)
- U4 pad GND1: unconnected-(U4-PadGND1) -> GND
- U4 pad GND2: unconnected-(U4-PadGND2) -> GND
- U4 pad RX+: unconnected-(U4-PadRX+) -> /Ethernet PHY/RXP
- U4 pad RX-: unconnected-(U4-PadRX-) -> /Ethernet PHY/RXN
- U4 pad RXCT: unconnected-(U4-PadRXCT) -> /VDDA_3V3
- U4 pad TX+: unconnected-(U4-PadTX+) -> /Ethernet PHY/TXP
- U4 pad TX-: unconnected-(U4-PadTX-) -> /Ethernet PHY/TXN
- U4 pad TXCT: unconnected-(U4-PadTXCT) -> /VDDA_3V3
- U4 pad Y+: unconnected-(U4-PadY+) -> Net-(R35-Pad1)
- U4 pad Y-: unconnected-(U4-PadY-) -> GND
- U5 pad 1: unconnected-(U5-VDD2A-Pad1) -> /VDDA_3V3
- U5 pad 10: unconnected-(U5-RXER/PHYAD0-Pad10) -> /Ethernet PHY/RXER/PHYADD0
- U5 pad 11: unconnected-(U5-CRS_DV/MODE2-Pad11) -> Net-(U5-CRS_DV/MODE2)
- U5 pad 12: unconnected-(U5-MDIO-Pad12) -> /Ethernet PHY/MDIO
- U5 pad 13: unconnected-(U5-MDC-Pad13) -> /Ethernet PHY/MDC
- U5 pad 15: unconnected-(U5-~{RST}-Pad15) -> Net-(U5-~{RST})
- U5 pad 16: unconnected-(U5-TXEN-Pad16) -> /Ethernet PHY/TXEN
- U5 pad 17: unconnected-(U5-TXD0-Pad17) -> /Ethernet PHY/TXD0
- U5 pad 18: unconnected-(U5-TXD1-Pad18) -> /Ethernet PHY/TXD1
- U5 pad 19: unconnected-(U5-VDD1A-Pad19) -> /VDDA_3V3
- U5 pad 2: unconnected-(U5-LED2/~{INTSEL}-Pad2) -> /Ethernet PHY/ETH_LINK_LED
- U5 pad 20: unconnected-(U5-TXN-Pad20) -> /Ethernet PHY/TXN
- U5 pad 21: unconnected-(U5-TXP-Pad21) -> /Ethernet PHY/TXP
- U5 pad 22: unconnected-(U5-RXN-Pad22) -> /Ethernet PHY/RXN
- U5 pad 23: unconnected-(U5-RXP-Pad23) -> /Ethernet PHY/RXP
- U5 pad 24: unconnected-(U5-RBIAS-Pad24) -> Net-(U5-RBIAS)
- U5 pad 25: unconnected-(U5-VSS-Pad25) -> GND
- U5 pad 3: unconnected-(U5-LED1/REGOFF-Pad3) -> /Ethernet PHY/ETH_ACT_LED
- U5 pad 5: unconnected-(U5-XTAL1/CLKIN-Pad5) -> Net-(U5-XTAL1/CLKIN)
- U5 pad 6: unconnected-(U5-VDDCR-Pad6) -> Net-(U5-VDDCR)
- U5 pad 7: unconnected-(U5-RXD1/MODE1-Pad7) -> Net-(U5-RXD1/MODE1)
- U5 pad 8: unconnected-(U5-RXD0/MODE0-Pad8) -> Net-(U5-RXD0/MODE0)
- U5 pad 9: unconnected-(U5-VDDIO-Pad9) -> VP3V3
- U8 pad 34: VBAT -> VP3V3
- U8 pad 35: VBAT -> VP3V3
- U8 pad 68: unconnected-(U8-GNSS_ANT-Pad68) -> Net-(U8-GNSS_ANT)
Other:
- board size 135 x 56 mm -> 148.8 x 78.8 mm
- board text removed: "NMEA2000"

Commit message: Power layout started
Parts:
- removed D3: 0R, Diode_SMD:D_0603_1608Metric
- added C36: 10uF, Capacitor_SMD:C_0603_1608Metric, F.Cu at (191.0, 54.2)
- added D14: D, Diode_SMD:D_1206_3216Metric, F.Cu at (192.0, 111.5)
- added D15: D, Diode_SMD:D_1206_3216Metric, F.Cu at (213.2, 109.8)
- R34: footprint Resistor_SMD:R_0201_0603Metric -> Resistor_SMD:R_0402_1005Metric
- R4, R5, R6, R7: footprint Resistor_SMD:R_0201_0603Metric -> Resistor_SMD:R_0603_1608Metric
- R40, R41, R42: footprint Resistor_SMD:R_0603_1608Metric -> Resistor_SMD:R_0402_1005Metric
- moved C19 247.0 mm to (230.0, 127.0), turned to -90 degrees
- moved R35 246.9 mm to (228.0, 127.0), turned to 90 degrees
- moved R36 246.8 mm to (226.0, 127.0), turned to 90 degrees
- moved C1 192.7 mm to (234.5, 69.8), turned to 90 degrees
- moved C2 191.5 mm to (232.8, 69.8), turned to 90 degrees
- moved C3 190.3 mm to (231.0, 69.8), turned to 90 degrees
- moved FB7 188.6 mm to (232.0, 72.3), turned to 180 degrees
- moved U6 174.6 mm to (229.5, 75.3), turned to 180 degrees
- moved R57 153.2 mm to (175.0, 112.6), turned to 180 degrees
- moved D12 148.8 mm to (175.0, 109.1), turned to -90 degrees
- moved R58 148.7 mm to (179.5, 112.5), turned to 180 degrees
- moved U15 148.3 mm to (177.2, 102.8), turned to -90 degrees
- moved C34 146.8 mm to (181.5, 101.0), turned to -90 degrees
- moved D11 144.2 mm to (179.5, 109.0), turned to -90 degrees
- moved U11 138.8 mm to (193.8, 97.1), turned to 90 degrees
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Connections:
- C1 pad 2: Net-(U2--VDC) -> GND
- C2 pad 2: Net-(U2--VDC) -> GND
- C3 pad 2: Net-(U2--VDC) -> GND
- D13 pad 1: /NMEA2000/CAN_L -> /NMEA2000/CAN_H
- D13 pad 2: /NMEA2000/CAN_H -> /NMEA2000/CAN_L
- D6 pad 1: Net-(U7-VCC) -> unconnected-(D6-K-Pad1)
- D6 pad 5: Net-(U7-I/O) -> Net-(U7-CLK)
- D6 pad 6: Net-(U7-CLK) -> Net-(U7-I/O)
- J1 pad 1: VP12V -> Net-(D14-A)
- J3 pad 1: /NMEA0183/TXP -> /NMEA0183/TXN
- J3 pad 2: /NMEA0183/TXN -> /NMEA0183/TXP
- J3 pad 3: /NMEA0183/RXP -> /NMEA0183/RXN
- J3 pad 4: /NMEA0183/RXN -> /NMEA0183/RXP
- J8 pad 4: VP12V -> Net-(D15-A)
- PoE+1 pad 1: /Power/VP_PoE -> unconnected-(PoE+1-Pad1)
- PoE-1 pad 1: /Power/VN_PoE -> unconnected-(PoE-1-Pad1)
- R55 pad 2: Net-(U2--VDC) -> GND
- TP1 pad 1: /Ethernet PHY/MDC -> unconnected-(TP1-Pad1)
- TP10 pad 1: VP3V3 -> unconnected-(TP10-Pad1)
- TP11 pad 1: VP5V -> unconnected-(TP11-Pad1)
- TP13 pad 1: /Power/VP_USB -> unconnected-(TP13-Pad1)
- TP14 pad 1: /Microcontroller/ESP_RXD0 -> unconnected-(TP14-Pad1)
- TP15 pad 1: /Microcontroller/ESP_TXD0 -> unconnected-(TP15-Pad1)
- TP16 pad 1: /Microcontroller/CH_DTR -> unconnected-(TP16-Pad1)
- TP17 pad 1: /Microcontroller/CH_RTS -> unconnected-(TP17-Pad1)
- TP18 pad 1: /Microcontroller/AIS_UART0_TX -> unconnected-(TP18-Pad1)
- TP19 pad 1: /Microcontroller/AIS_UART0_RX -> unconnected-(TP19-Pad1)
- TP2 pad 1: /Ethernet PHY/MDIO -> unconnected-(TP2-Pad1)
- TP20 pad 1: /Microcontroller/CAN_RX -> unconnected-(TP20-Pad1)
- TP21 pad 1: /Microcontroller/CAN_TX -> unconnected-(TP21-Pad1)
- TP3 pad 1: /Microcontroller/NMEA0183_TX -> unconnected-(TP3-Pad1)
- TP4 pad 1: /Microcontroller/NMEA0183_RX -> unconnected-(TP4-Pad1)
- TP5 pad 1: /Microcontroller/MODEM_PWR -> unconnected-(TP5-Pad1)
- TP6 pad 1: /Microcontroller/MODEM_DTR -> unconnected-(TP6-Pad1)
- TP7 pad 1: /Microcontroller/MODEM_TX -> unconnected-(TP7-Pad1)
- TP8 pad 1: /Microcontroller/MODEM_RX -> unconnected-(TP8-Pad1)
- TP9 pad 1: VP12V -> unconnected-(TP9-Pad1)
- U12 pad 16: /USB to Serial/VP3V3 -> VP3V3
- U2 pad 3: Net-(U2--VDC) -> GND
Routing:
- net /Ethernet PHY/TXD1: track 0.00 -> 50.5 mm
- net /Ethernet PHY/TXEN: track 0.00 -> 48.6 mm
- net /Ethernet PHY/TXD0: track 0.00 -> 47.8 mm
- net /Ethernet PHY/TXN: track 0.00 -> 20.8 mm
- net /Power/VN_PoE: track 0.00 -> 20.8 mm
- net /Ethernet PHY/TXP: track 0.00 -> 16.6 mm
- net /Power/VP_PoE: track 0.00 -> 16.4 mm
- net /NMEA0183/RXP: track 0.00 -> 12.3 mm
- net /NMEA0183/TXN: track 0.00 -> 12.1 mm
- net /NMEA0183/TXP: track 0.00 -> 11.1 mm
- net /NMEA0183/RXN: track 0.00 -> 11.1 mm
- net /Ethernet PHY/RXER/PHYADD0: track 0.00 -> 10.4 mm, vias 0 -> 2
- net /Ethernet PHY/RXD0/MODE0: track 0.00 -> 10.1 mm, vias 0 -> 2
- net /Ethernet PHY/RXD1/MODE1: track 0.00 -> 9.31 mm
- net /Ethernet PHY/CRS_DV/MODE2: track 0.00 -> 9.18 mm
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Other:
- board text added: "BRD_PWR"
- board text added: "NETWORK"
- board text added: "STATUS"
