File: nmea2000.kicad_sch (KiCad schematic)
At the start: 4 parts, among them U16 TJA1051T-3

Commit message: Power layout started
Connections:
- net CAN_H: now also D13.1 (A1); no longer D13.2 (A2)
- net CAN_L: now also D13.2 (A2); no longer D13.1 (A1)
Changed lines of the file:
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@@
 	)
 	(junction
-		(at 226.06 111.76)
+		(at 226.06 106.68)
 		(diameter 0)
 		(color 0 0 0 0)
@@
 	)
 	(junction
-		(at 203.2 106.68)
-		(diameter 0)
-		(color 0 0 0 0)
-	)
-	(junction
 		(at 127 81.28)
 		(diameter 0)
@@
 	)
 	(junction
+		(at 203.2 111.76)
+		(diameter 0)
+		(color 0 0 0 0)
+	)
+	(junction
 		(at 127 133.35)
 		(diameter 0)
@@
 	(wire
 		(pts
-			(xy 226.06 111.76) (xy 226.06 129.54)
-		)
-		(stroke
-			(width 0)
-			(type default)
-		)
-	)
-	(wire
-		(pts
 			(xy 127 128.27) (xy 127 133.35)
 		)
@@
 	(wire
 		(pts
-			(xy 181.61 111.76) (xy 226.06 111.76)
+			(xy 181.61 111.76) (xy 203.2 111.76)
 		)
 		(stroke
@@
 	(wire
 		(pts
-			(xy 203.2 129.54) (xy 203.2 106.68)
-		)
-		(stroke
-			(width 0)
-			(type default)
-		)
-	)
-	(wire
-		(pts
 			(xy 127 114.3) (xy 127 120.65)
 		)
@@
 	(wire
 		(pts
-			(xy 203.2 106.68) (xy 248.92 106.68)
-		)
-		(stroke
-			(width 0)
-			(type default)
-		)
-	)
-	(wire
-		(pts
 			(xy 127 81.28) (xy 144.78 81.28)
 		)
@@
 	(wire
 		(pts
+			(xy 226.06 106.68) (xy 248.92 106.68)
+		)
+		(stroke
+			(width 0)
+			(type default)
+		)
+	)
+	(wire
+		(pts
 			(xy 100.33 104.14) (xy 132.08 104.14)
 		)
@@
 	(wire
 		(pts
+			(xy 203.2 111.76) (xy 203.2 129.54)
+		)
+		(stroke
+			(width 0)
+			(type default)
+		)
+	)
+	(wire
+		(pts
 			(xy 100.33 106.68) (xy 132.08 106.68)
 		)
@@
 	(wire
 		(pts
-			(xy 226.06 111.76) (xy 248.92 111.76)
-		)
-		(stroke
-			(width 0)
-			(type default)
-		)
-	)
-	(wire
-		(pts
 			(xy 144.78 81.28) (xy 158.75 81.28)
 		)
@@
 	(wire
 		(pts
-			(xy 181.61 106.68) (xy 203.2 106.68)
+			(xy 181.61 106.68) (xy 226.06 106.68)
 		)
 		(stroke
@@
 	(wire
 		(pts
+			(xy 226.06 106.68) (xy 226.06 129.54)
+		)
+		(stroke
+			(width 0)
+			(type default)
+		)
+	)
+	(wire
+		(pts
 			(xy 100.33 81.28) (xy 127 81.28)
 		)
 		(stroke
+			(width 0)
+			(type default)
+		)
+	)
+	(wire
+		(pts
+			(xy 203.2 111.76) (xy 248.92 111.76)
+		)
+		(stroke
